File: src/pcb/Anchor/Anchor PCB V1.sch (EAGLE design)
At the start: 89 parts, among them IC1 ENC28J60-I_SS, IC2 TPS23750PWP, IC3 MIC5219-3.3YM5-TR, IC4 DWM1000, J1 0826-1X1T-GJ-F, J2 105017-0001, Q1 32 MHz, Q2 SUD06N10-225L, U1 ATSAMD21G-A, Y1 25 MHz

Commit message: Changed footprint 33µH
Parts:
- L2: device inductors:DR73 -> wurth_elektronik_passive_rev16d:WE-PD_1260/1245/1280/1210
Changed lines of the file:
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@@
 <layers>
 <layer number="1" name="Top" color="4" fill="1" visible="no" active="no"/>
+<layer number="2" name="Route2" color="1" fill="3" visible="no" active="no"/>
+<layer number="3" name="Route3" color="4" fill="3" visible="no" active="no"/>
+<layer number="4" name="Route4" color="1" fill="4" visible="no" active="no"/>
+<layer number="5" name="Route5" color="4" fill="4" visible="no" active="no"/>
+<layer number="6" name="Route6" color="1" fill="8" visible="no" active="no"/>
+<layer number="7" name="Route7" color="4" fill="8" visible="no" active="no"/>
+<layer number="8" name="Route8" color="1" fill="2" visible="no" active="no"/>
+<layer number="9" name="Route9" color="4" fill="2" visible="no" active="no"/>
+<layer number="10" name="Route10" color="1" fill="7" visible="no" active="no"/>
+<layer number="11" name="Route11" color="4" fill="7" visible="no" active="no"/>
+<layer number="12" name="Route12" color="1" fill="5" visible="no" active="no"/>
+<layer number="13" name="Route13" color="4" fill="5" visible="no" active="no"/>
+<layer number="14" name="Route14" color="1" fill="6" visible="no" active="no"/>
+<layer number="15" name="Route15" color="4" fill="6" visible="no" active="no"/>
 <layer number="16" name="Bottom" color="1" fill="1" visible="no" active="no"/>
 <layer number="17" name="Pads" color="2" fill="1" visible="no" active="no"/>
@@
 <part name="Q2" library="transistor-power" library_urn="urn:adsk.eagle:library:400" deviceset="N-HEXFET_?-*" device="SOT323" package3d_urn="urn:adsk.eagle:package:29522/2" technology="IRLL014N" value="SUD06N10-225L"/>
 <part name="R10" library="rcl" library_urn="urn:adsk.eagle:library:334" deviceset="R-EU_" device="R0805" package3d_urn="urn:adsk.eagle:package:23553/2" value="10 Ω"/>
-<part name="L2" library="inductors" library_urn="urn:adsk.eagle:library:243" deviceset="DR73" device="" package3d_urn="urn:adsk.eagle:package:15123/1" value="33 µH"/>
+<part name="L2" library="wurth_elektronik_passive_rev16d" deviceset="WE-PD" device="_1260/1245/1280/1210" value="33 µH"/>
 <part name="GND19" library="supply1" library_urn="urn:adsk.eagle:library:371" deviceset="GND" device=""/>
 <part name="D2" library="shottky" deviceset="BAS70-05" device="DPAK" package3d_urn="urn:adsk.eagle:package:28765/1" value="6CWQ10FN"/>

Commit message: Update anchor wrong footprints
Parts:
- C23: device rcl:CPOL-EUUD-5X5,8 -> rcl:CPOL-EUUD-6,3X7,7
Changed lines of the file:
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@@
 <grid distance="0.05" unitdist="inch" unit="inch" style="lines" multiple="1" display="no" altdistance="0.01" altunitdist="inch" altunit="inch"/>
 <layers>
-<layer number="1" name="Top" color="4" fill="1" visible="no" active="no"/>
-<layer number="2" name="Route2" color="1" fill="3" visible="no" active="no"/>
-<layer number="3" name="Route3" color="4" fill="3" visible="no" active="no"/>
-<layer number="4" name="Route4" color="1" fill="4" visible="no" active="no"/>
-<layer number="5" name="Route5" color="4" fill="4" visible="no" active="no"/>
-<layer number="6" name="Route6" color="1" fill="8" visible="no" active="no"/>
-<layer number="7" name="Route7" color="4" fill="8" visible="no" active="no"/>
-<layer number="8" name="Route8" color="1" fill="2" visible="no" active="no"/>
-<layer number="9" name="Route9" color="4" fill="2" visible="no" active="no"/>
-<layer number="10" name="Route10" color="1" fill="7" visible="no" active="no"/>
-<layer number="11" name="Route11" color="4" fill="7" visible="no" active="no"/>
-<layer number="12" name="Route12" color="1" fill="5" visible="no" active="no"/>
-<layer number="13" name="Route13" color="4" fill="5" visible="no" active="no"/>
-<layer number="14" name="Route14" color="1" fill="6" visible="no" active="no"/>
-<layer number="15" name="Route15" color="4" fill="6" visible="no" active="no"/>
-<layer number="16" name="Bottom" color="1" fill="1" visible="no" active="no"/>
-<layer number="17" name="Pads" color="2" fill="1" visible="no" active="no"/>
-<layer number="18" name="Vias" color="2" fill="1" visible="no" active="no"/>
-<layer number="19" name="Unrouted" color="6" fill="1" visible="no" active="no"/>
-<layer number="20" name="Dimension" color="24" fill="1" visible="no" active="no"/>
-<layer number="21" name="tPlace" color="7" fill="1" visible="no" active="no"/>
-<layer number="22" name="bPlace" color="7" fill="1" visible="no" active="no"/>
-<layer number="23" name="tOrigins" color="15" fill="1" visible="no" active="no"/>
-<layer number="24" name="bOrigins" color="15" fill="1" visible="no" active="no"/>
-<layer number="25" name="tNames" color="7" fill="1" visible="no" active="no"/>
-<layer number="26" name="bNames" color="7" fill="1" visible="no" active="no"/>
-<layer number="27" name="tValues" color="7" fill="1" visible="no" active="no"/>
-<layer number="28" name="bValues" color="7" fill="1" visible="no" active="no"/>
+<layer number="1" name="Top" color="4" fill="1" visible="yes" active="no"/>
+<layer number="2" name="Route2" color="16" fill="1" visible="yes" active="no"/>
+<layer number="3" name="Route3" color="17" fill="1" visible="yes" active="no"/>
+<layer number="4" name="Route4" color="18" fill="1" visible="yes" active="no"/>
+<layer number="5" name="Route5" color="19" fill="1" visible="yes" active="no"/>
+<layer number="6" name="Route6" color="25" fill="1" visible="yes" active="no"/>
+<layer number="7" name="Route7" color="26" fill="1" visible="yes" active="no"/>
+<layer number="8" name="Route8" color="27" fill="1" visible="yes" active="no"/>
+<layer number="9" name="Route9" color="28" fill="1" visible="yes" active="no"/>
+<layer number="10" name="Route10" color="29" fill="1" visible="yes" active="no"/>
+<layer number="11" name="Route11" color="30" fill="1" visible="yes" active="no"/>
+<layer number="12" name="Route12" color="20" fill="1" visible="yes" active="no"/>
+<layer number="13" name="Route13" color="21" fill="1" visible="yes" active="no"/>
+<layer number="14" name="Route14" color="22" fill="1" visible="yes" active="no"/>
+<layer number="15" name="Route15" color="23" fill="1" visible="yes" active="no"/>
+<layer number="16" name="Bottom" color="1" fill="1" visible="yes" active="no"/>
+<layer number="17" name="Pads" color="2" fill="1" visible="yes" active="no"/>
+<layer number="18" name="Vias" color="2" fill="1" visible="yes" active="no"/>
+<layer number="19" name="Unrouted" color="6" fill="1" visible="yes" active="no"/>
+<layer number="20" name="Dimension" color="24" fill="1" visible="yes" active="no"/>
+<layer number="21" name="tPlace" color="7" fill="1" visible="yes" active="no"/>
+<layer number="22" name="bPlace" color="7" fill="1" visible="yes" active="no"/>
+<layer number="23" name="tOrigins" color="15" fill="1" visible="yes" active="no"/>
+<layer number="24" name="bOrigins" color="15" fill="1" visible="yes" active="no"/>
+<layer number="25" name="tNames" color="7" fill="1" visible="yes" active="no"/>
+<layer number="26" name="bNames" color="7" fill="1" visible="yes" active="no"/>
+<layer number="27" name="tValues" color="7" fill="1" visible="yes" active="no"/>
+<layer number="28" name="bValues" color="7" fill="1" visible="yes" active="no"/>
 <layer number="29" name="tStop" color="7" fill="3" visible="no" active="no"/>
 <layer number="30" name="bStop" color="7" fill="6" visible="no" active="no"/>
@@
 <layer number="35" name="tGlue" color="7" fill="4" visible="no" active="no"/>
 <layer number="36" name="bGlue" color="7" fill="5" visible="no" active="no"/>
-<layer number="37" name="tTest" color="7" fill="1" visible="no" active="no"/>
-<layer number="38" name="bTest" color="7" fill="1" visible="no" active="no"/>
+<layer number="37" name="tTest" color="7" fill="1" visible="yes" active="no"/>
+<layer number="38" name="bTest" color="7" fill="1" visible="yes" active="no"/>
 <layer number="39" name="tKeepout" color="4" fill="11" visible="no" active="no"/>
 <layer number="40" name="bKeepout" color="1" fill="11" visible="no" active="no"/>
@@
 <layer number="44" name="Drills" color="7" fill="1" visible="no" active="no"/>
 <layer number="45" name="Holes" color="7" fill="1" visible="no" active="no"/>
-<layer number="46" name="Milling" color="3" fill="1" visible="no" active="no"/>
-<layer number="47" name="Measures" color="7" fill="1" visible="no" active="no"/>
-<layer number="48" name="Document" color="7" fill="1" visible="no" active="no"/>
-<layer number="49" name="Reference" color="7" fill="1" visible="no" active="no"/>
-<layer number="50" name="dxf" color="7" fill="1" visible="no" active="no"/>
-<layer number="51" name="tDocu" color="7" fill="1" visible="no" active="no"/>
-<layer number="52" name="bDocu" color="7" fill="1" visible="no" active="no"/>
-<layer number="53" name="tGND_GNDA" color="7" fill="9" visible="no" active="no"/>
-<layer number="54" name="bGND_GNDA" color="1" fill="9" visible="no" active="no"/>
-<layer number="56" name="wert" color="7" fill="1" visible="no" active="no"/>
-<layer number="57" name="tCAD" color="7" fill="1" visible="no" active="no"/>
-<layer number="59" name="tCarbon" color="7" fill="1" visible="no" active="no"/>
-<layer number="60" name="bCarbon" color="7" fill="1" visible="no" active="no"/>
+<layer number="46" name="Milling" color="3" fill="1" visible="yes" active="no"/>
+<layer number="47" name="Measures" color="7" fill="1" visible="yes" active="no"/>
+<layer number="48" name="Document" color="7" fill="1" visible="yes" active="no"/>
+<layer number="49" name="Reference" color="7" fill="1" visible="yes" active="no"/>
+<layer number="50" name="dxf" color="7" fill="1" visible="yes" active="no"/>
+<layer number="51" name="tDocu" color="7" fill="1" visible="yes" active="no"/>
+<layer number="52" name="bDocu" color="7" fill="1" visible="yes" active="no"/>
+<layer number="53" name="tGND_GNDA" color="7" fill="9" visible="yes" active="no"/>
+<layer number="54" name="bGND_GNDA" color="1" fill="9" visible="yes" active="no"/>
+<layer number="56" name="wert" color="7" fill="1" visible="yes" active="no"/>
+<layer number="57" name="tCAD" color="7" fill="1" visible="yes" active="no"/>
+<layer number="59" name="tCarbon" color="7" fill="1" visible="yes" active="no"/>
+<layer number="60" name="bCarbon" color="7" fill="1" visible="yes" active="no"/>
 <layer number="88" name="SimResults" color="9" fill="1" visible="yes" active="yes"/>
 <layer number="89" name="SimProbes" color="9" fill="1" visible="yes" active="yes"/>
@@
 <part name="C20" library="rcl" library_urn="urn:adsk.eagle:library:334" deviceset="C-EU" device="C0805" package3d_urn="urn:adsk.eagle:package:23617/2" value="10 µF (6.3V)"/>
 <part name="C21" library="rcl" library_urn="urn:adsk.eagle:library:334" deviceset="C-EU" device="C0805" package3d_urn="urn:adsk.eagle:package:23617/2" value="10 µF (6.3V)"/>
-<part name="C23" library="rcl" library_urn="urn:adsk.eagle:library:334" deviceset="CPOL-EU" device="UD-5X5,8" package3d_urn="urn:adsk.eagle:package:23470/1" value="100 µF (6.3V)"/>
+<part name="C23" library="rcl" library_urn="urn:adsk.eagle:library:334" deviceset="CPOL-EU" device="UD-6,3X7,7" package3d_urn="urn:adsk.eagle:package:23472/1" value="100 µF (6.3V)"/>
 <part name="GND22" library="supply1" library_urn="urn:adsk.eagle:library:371" deviceset="GND" device=""/>
 <part name="GND23" library="supply1" library_urn="urn:adsk.eagle:library:371" deviceset="GND" device=""/>

Commit message: Added backups for schematic and board
Parts:
- D3: device SparkFun-LED:LED-BLUE1206 -> led:LEDCHIP-LED0805
- D4, D6: device SparkFun-LED:LED-YELLOWLILYPAD -> led:LEDCHIP-LED0805
- D5, D7: device SparkFun-LED:LED-GREENLILYPAD -> led:LEDCHIP-LED0805
Connections:
- new net RXLED_MC: D5.C, U1.PB3-A6
- new net TXLED_MC: D4.C, U1.PA27
- net RX_MC: now also JP4.1; no longer D5.C, JP4.2, U1.PB23
- net TX_MC: now also JP4.2; no longer D4.C, JP4.1, U1.PB22
Other:
- moved on the sheet: JP2
Changed lines of the file:
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@@
 <part name="GND43" library="supply1" library_urn="urn:adsk.eagle:library:371" deviceset="GND" device=""/>
 <part name="P+13" library="supply1" library_urn="urn:adsk.eagle:library:371" deviceset="VCC" device="" value="3.3V"/>
-<part name="D3" library="SparkFun-LED" deviceset="LED-BLUE" device="1206" value="POWER"/>
+<part name="D3" library="led" library_urn="urn:adsk.eagle:library:259" deviceset="LED" device="CHIP-LED0805" package3d_urn="urn:adsk.eagle:package:15818/2" value="POWER"/>
 <part name="R3" library="rcl" library_urn="urn:adsk.eagle:library:334" deviceset="R-EU_" device="R0805" package3d_urn="urn:adsk.eagle:package:23553/2" value="470 Ω"/>
 <part name="GND29" library="supply1" library_urn="urn:adsk.eagle:library:371" deviceset="GND" device=""/>
 <part name="R14" library="rcl" library_urn="urn:adsk.eagle:library:334" deviceset="R-EU_" device="R0805" package3d_urn="urn:adsk.eagle:package:23553/2" value="270 Ω"/>
 <part name="R26" library="rcl" library_urn="urn:adsk.eagle:library:334" deviceset="R-EU_" device="R0805" package3d_urn="urn:adsk.eagle:package:23553/2" value="220 Ω"/>
-<part name="D4" library="SparkFun-LED" deviceset="LED-YELLOW" device="LILYPAD" value="TX"/>
-<part name="D5" library="SparkFun-LED" deviceset="LED-GREEN" device="LILYPAD" value="RX"/>
+<part name="D4" library="led" library_urn="urn:adsk.eagle:library:259" deviceset="LED" device="CHIP-LED0805" package3d_urn="urn:adsk.eagle:package:15818/2" value="TX"/>
+<part name="D5" library="led" library_urn="urn:adsk.eagle:library:259" deviceset="LED" device="CHIP-LED0805" package3d_urn="urn:adsk.eagle:package:15818/2" value="RX"/>
 <part name="IC4" library="DWM1000" deviceset="DWM1000" device=""/>
 <part name="P+14" library="supply1" library_urn="urn:adsk.eagle:library:371" deviceset="VCC" device="" value="3.3V"/>
@@
 <part name="R28" library="rcl" library_urn="urn:adsk.eagle:library:334" deviceset="R-EU_" device="R0805" package3d_urn="urn:adsk.eagle:package:23553/2" value="270 Ω"/>
 <part name="R29" library="rcl" library_urn="urn:adsk.eagle:library:334" deviceset="R-EU_" device="R0805" package3d_urn="urn:adsk.eagle:package:23553/2" value="220 Ω"/>
-<part name="D6" library="SparkFun-LED" deviceset="LED-YELLOW" device="LILYPAD" value="TX"/>
-<part name="D7" library="SparkFun-LED" deviceset="LED-GREEN" device="LILYPAD" value="RX"/>
+<part name="D6" library="led" library_urn="urn:adsk.eagle:library:259" deviceset="LED" device="CHIP-LED0805" package3d_urn="urn:adsk.eagle:package:15818/2" value="TX"/>
+<part name="D7" library="led" library_urn="urn:adsk.eagle:library:259" deviceset="LED" device="CHIP-LED0805" package3d_urn="urn:adsk.eagle:package:15818/2" value="RX"/>
 <part name="P+15" library="supply1" library_urn="urn:adsk.eagle:library:371" deviceset="VCC" device="" value="3.3V"/>
 <part name="GND31" library="supply1" library_urn="urn:adsk.eagle:library:371" deviceset="GND" device=""/>
@@
 <instance part="D3" gate="G$1" x="-254" y="-24.13" smashed="yes">
 <attribute name="NAME" x="-257.429" y="-28.702" size="1.778" layer="95" font="vector" rot="R90"/>
-<attribute name="VALUE" x="-252.095" y="-28.702" size="1.778" layer="96" font="vector" rot="R90" align="top-left"/>
 </instance>
 <instance part="R3" gate="G$1" x="-254" y="-15.24" smashed="yes" rot="R90">
@@
 <instance part="D4" gate="G$1" x="-243.84" y="-24.13" smashed="yes">
 <attribute name="NAME" x="-247.269" y="-28.702" size="1.778" layer="95" font="vector" rot="R90"/>
-<attribute name="VALUE" x="-241.935" y="-28.702" size="1.778" layer="96" font="vector" rot="R90" align="top-left"/>
 </instance>
 <instance part="D5" gate="G$1" x="-233.68" y="-24.13" smashed="yes">
 <attribute name="NAME" x="-237.109" y="-28.702" size="1.778" layer="95" font="vector" rot="R90"/>
-<attribute name="VALUE" x="-231.775" y="-28.702" size="1.778" layer="96" font="vector" rot="R90" align="top-left"/>
 </instance>
 <instance part="IC4" gate="G$1" x="-17.78" y="91.44" smashed="yes">
@@
 <instance part="D6" gate="G$1" x="-12.7" y="26.67" smashed="yes">
 <attribute name="NAME" x="-16.129" y="22.098" size="1.778" layer="95" font="vector" rot="R90"/>
-<attribute name="VALUE" x="-10.795" y="22.098" size="1.778" layer="96" font="vector" rot="R90" align="top-left"/>
 </instance>
 <instance part="D7" gate="G$1" x="-2.54" y="26.67" smashed="yes">
 <attribute name="NAME" x="-5.969" y="22.098" size="1.778" layer="95" font="vector" rot="R90"/>
-<attribute name="VALUE" x="-0.635" y="22.098" size="1.778" layer="96" font="vector" rot="R90" align="top-left"/>
 </instance>
 <instance part="P+15" gate="VCC" x="-2.54" y="48.26" smashed="yes">
@@
 <attribute name="VALUE" x="-106.68" y="97.79" size="1.778" layer="96" rot="R90" align="center-left"/>
 </instance>
-<instance part="JP2" gate="A" x="-210.82" y="69.85" smashed="yes" rot="R270">
-<attribute name="NAME" x="-210.82" y="71.12" size="1.778" layer="95"/>
-<attribute name="VALUE" x="-210.82" y="64.135" size="1.778" layer="96"/>
-</instance>
-<instance part="GND8" gate="1" x="-218.44" y="62.23" smashed="yes">
-<attribute name="VALUE" x="-215.9" y="60.96" size="1.778" layer="96" rot="R180"/>
-</instance>
-<instance part="P+6" gate="VCC" x="-218.44" y="73.66" smashed="yes">
-<attribute name="VALUE" x="-215.9" y="76.2" size="1.778" layer="96" rot="R180"/>
+<instance part="JP2" gate="A" x="-210.82" y="72.39" smashed="yes" rot="R270">
+<attribute name="NAME" x="-210.82" y="73.66" size="1.778" layer="95"/>
+<attribute name="VALUE" x="-210.82" y="66.675" size="1.778" layer="96"/>
+</instance>
+<instance part="GND8" gate="1" x="-218.44" y="64.77" smashed="yes">
+<attribute name="VALUE" x="-215.9" y="63.5" size="1.778" layer="96" rot="R180"/>
+</instance>
+<instance part="P+6" gate="VCC" x="-218.44" y="76.2" smashed="yes">
+<attribute name="VALUE" x="-215.9" y="78.74" size="1.778" layer="96" rot="R180"/>
 </instance>
 <instance part="JP3" gate="A" x="-360.68" y="29.21" smashed="yes" rot="R270">
@@
 <pinref part="GND8" gate="1" pin="GND"/>
 <pinref part="JP2" gate="A" pin="2"/>
-<wire x1="-218.44" y1="64.77" x2="-218.44" y2="67.31" width="0.1524" layer="91"/>
-<wire x1="-218.44" y1="67.31" x2="-213.36" y2="67.31" width="0.1524" layer="91"/>
+<wire x1="-218.44" y1="67.31" x2="-218.44" y2="69.85" width="0.1524" layer="91"/>
+<wire x1="-218.44" y1="69.85" x2="-213.36" y2="69.85" width="0.1524" layer="91"/>
 </segment>
 <segment>
@@
 <segment>
 <pinref part="JP2" gate="A" pin="1"/>
-<wire x1="-213.36" y1="69.85" x2="-218.44" y2="69.85" width="0.1524" layer="91"/>
-<wire x1="-218.44" y1="69.85" x2="-218.44" y2="71.12" width="0.1524" layer="91"/>
+<wire x1="-213.36" y1="72.39" x2="-218.44" y2="72.39" width="0.1524" layer="91"/>
+<wire x1="-218.44" y1="72.39" x2="-218.44" y2="73.66" width="0.1524" layer="91"/>
 <pinref part="P+6" gate="VCC" pin="VCC"/>
 </segment>
@@
 </segment>
 </net>
-<net name="RX_MC" class="0">
-<segment>
-<pinref part="U1" gate="G$1" pin="D0/RX"/>
-<wire x1="-195.58" y1="-33.02" x2="-195.58" y2="-35.56" width="0.1524" layer="91"/>
-<label x="-195.58" y="-35.56" size="1.778" layer="95" rot="R270" xref="yes"/>
-</segment>
+<net name="RXLED_MC" class="0">
 <segment>
 <pinref part="D5" gate="G$1" pin="C"/>
@@
 </segment>
 <segment>
-<pinref part="U1" gate="G$1" pin="PB23"/>
-<wire x1="-160.02" y1="48.26" x2="-160.02" y2="50.8" width="0.1524" layer="91"/>
-<label x="-160.02" y="50.8" size="1.778" layer="95" rot="R90" xref="yes"/>
-</segment>
-<segment>
-<pinref part="JP4" gate="A" pin="2"/>
-<wire x1="-232.41" y1="-59.69" x2="-246.38" y2="-59.69" width="0.1524" layer="91"/>
-<label x="-246.38" y="-59.69" size="1.778" layer="95" rot="R180" xref="yes"/>
-</segment>
-</net>
-<net name="TX_MC" class="0">
-<segment>
-<pinref part="U1" gate="G$1" pin="D1/TX"/>
-<wire x1="-200.66" y1="-33.02" x2="-200.66" y2="-35.56" width="0.1524" layer="91"/>
-<label x="-200.66" y="-35.56" size="1.778" layer="95" rot="R270" xref="yes"/>
-</segment>
+<pinref part="U1" gate="G$1" pin="PB3-A6"/>
+<wire x1="-210.82" y1="48.26" x2="-210.82" y2="49.53" width="0.1524" layer="91"/>
+<label x="-210.82" y="49.53" size="1.778" layer="95" rot="R90" xref="yes"/>
+</segment>
+</net>
+<net name="TXLED_MC" class="0">
 <segment>
 <pinref part="D4" gate="G$1" pin="C"/>
@@
 </segment>
 <segment>
-<pinref part="U1" gate="G$1" pin="PB22"/>
-<wire x1="-154.94" y1="48.26" x2="-154.94" y2="50.8" width="0.1524" layer="91"/>
-<label x="-154.94" y="50.8" size="1.778" layer="95" rot="R90" xref="yes"/>
-</segment>
-<segment>
-<pinref part="JP4" gate="A" pin="1"/>
-<wire x1="-232.41" y1="-57.15" x2="-234.95" y2="-57.15" width="0.1524" layer="91"/>
-<label x="-234.95" y="-57.15" size="1.778" layer="95" rot="R180" xref="yes"/>
+<pinref part="U1" gate="G$1" pin="PA27"/>
+<wire x1="-165.1" y1="48.26" x2="-165.1" y2="53.34" width="0.1524" layer="91"/>
+<label x="-165.1" y="53.34" size="1.778" layer="95" rot="R90" xref="yes"/>
 </segment>
 </net>
@@
 </segment>
 </net>
+<net name="TX_MC" class="0">
+<segment>
+<pinref part="U1" gate="G$1" pin="D1/TX"/>
+<wire x1="-200.66" y1="-33.02" x2="-200.66" y2="-35.56" width="0.1524" layer="91"/>
+<label x="-200.66" y="-35.56" size="1.778" layer="95" rot="R270" xref="yes"/>
+</segment>
+<segment>
+<pinref part="JP4" gate="A" pin="2"/>
+<wire x1="-232.41" y1="-59.69" x2="-236.22" y2="-59.69" width="0.1524" layer="91"/>
+<label x="-236.22" y="-59.69" size="1.778" layer="95" rot="R180" xref="yes"/>
+</segment>
+</net>
+<net name="RX_MC" class="0">
+<segment>
+<pinref part="U1" gate="G$1" pin="D0/RX"/>
+<wire x1="-195.58" y1="-33.02" x2="-195.58" y2="-35.56" width="0.1524" layer="91"/>
+<label x="-195.58" y="-35.56" size="1.778" layer="95" rot="R270" xref="yes"/>
+</segment>
+<segment>
+<pinref part="JP4" gate="A" pin="1"/>
+<wire x1="-232.41" y1="-57.15" x2="-247.65" y2="-57.15" width="0.1524" layer="91"/>
+<label x="-247.65" y="-57.15" size="1.778" layer="95" rot="R180" xref="yes"/>
+</segment>
+</net>

Commit message: Solving connection problems
Connections:
- net MISO2_MC renamed MISO2_DWM
- net MOSI2_MC renamed MOSI2_DWM
- net SCK2_MC renamed SCK2_DWM
- net GND: now also D6.C, D7.C
- net IRQ: now also U1.D7
- net RXLED_DWM: now also R29.2; no longer D7.C
- net TXLED_DWM: now also R28.2; no longer D6.C
- net VCC: no longer R28.2, R29.2
Other:
- moved on the sheet: D6, D7, R28, R29
